File: RaspiLink/RaspiLink_bk1.brd (EAGLE design)
At the start: 65 x 55.9 mm, 21 parts, among them J1 SSM-120-S-SV, J2 SSM-120-S-SV, Q1 MOSFET-NCHANNELBSS123LT1G, Q2 MOSFET-NCHANNELBSS123LT1G, X1 SSW-120-02-S-D, X2 SSW-104-02-S-S

Commit message: joystick for crane
Parts:
- removed U$2: (no value), holes:3,0
- removed X2: SSW-104-02-S-S, con-samtec:SSW-104-02-S-S
- added X4: SSW-108-02-S-D, con-samtec:SSW-108-02-S-D
- moved R4 17.0 mm to (43.3, 49.6), turned to 270 degrees
- moved Q2 12.1 mm to (39.4, 49.6), turned to 270 degrees
- moved R2 10.4 mm to (43.3, 44.8), turned to 90 degrees
- moved R3 7.81 mm to (35.6, 49.6), turned to 90 degrees
- moved Q1 6.53 mm to (39.4, 44.8), turned to 270 degrees
- moved R1 5.85 mm to (35.6, 44.8), turned to 90 degrees
Connections:
- new net CM_RXD_1: J2.17
- new net CM_RXD_2: J2.10
- new net CM_TXD_1: J2.16
- new net CM_TXD_2: J2.9
- new net GPIO10_MOSI: X1.19
- new net GPIO11_CLK: X1.23
- new net GPIO17: X1.11
- new net GPIO18_PWM: X1.12
- new net GPIO22: X1.15
- new net GPIO23: X1.16
- new net GPIO24: X1.18
- new net GPIO25: X1.22
- new net GPIO27: X1.13
- new net GPIO4: X1.7
- new net GPIO7_CE1: X1.26
- new net GPIO8_CE0: X1.24
- new net GPIO9_MISO: X1.21
- net +3.3V: now also X1.1, X4.1; no longer X2.1
- net +5V: now also X4.2
- net GND: no longer X2.2
- net I2C_SCL: no longer X2.4
- net I2C_SDA: no longer X2.3
Routing:
- net VCC: track 102.8 -> 14.6 mm, vias 1 -> 0
- net I2C_SCL: track 81.9 -> 0.00 mm, vias 1 -> 0
- net I2C_SDA: track 81.3 -> 0.00 mm, vias 1 -> 0
- net +3.3V: track 73.1 -> 154.3 mm, vias 1 -> 5
- net CM_RX: track 61.6 -> 0.00 mm, vias 2 -> 0
- net +5V: track 63.6 -> 124.1 mm
- net CM_TX: track 51.4 -> 3.06 mm, vias 2 -> 0
- net GND: track 177.7 -> 152.6 mm
- net N$1: track 24.5 -> 0.00 mm
- net PI_RX: track 18.6 -> 28.3 mm
- net PI_TX: track 27.1 -> 32.6 mm, vias 2 -> 0
Other:
- outline, holes or cut-outs redrawn
